Commit message: Updated repository with latest local changes

File: my_hexacopter/urdf/gazebo_control.xacro (robot description, xacro)
@@ -1,5 +1,4 @@
 <?xml version='1.0'?>
 <robot xmlns:xacro="http://www.ros.org/wiki/xacro">
-    <!-- This part tells the ros2 controller what to actuate, how to actuate-->
     <ros2_control name="GazeboSystem" type="system">
         <hardware>
@@ -22,5 +21,4 @@
         </joint>
     </ros2_control>
-    <!-- This part tells Gazebo to use ros2_control-->
     <gazebo>
         <plugin name="gazebo_ros2_control" filename="libgazebo_ros2_control.so">

File: my_hexacopter/urdf/robot_arm.xacro (robot description, xacro)
@@ -2,13 +2,4 @@
 <robot name="robot_arm" xmlns:xacro="http://ros.org/wiki/xacro">
   <xacro:include filename="$(find my_hexacopter)/urdf/gazebo_control.xacro"/>
-  <!--<xacro:include filename="$(find my_hexacopter)/urdf/sensors.xacro"/>
-  <xacro:include filename="$(find my_hexacopter)/urdf/my_hexacopter_simple.xacro"/>-->
-  <!-- Fixed Joint to Connect Base Link to Hexacopter
-  <joint name="hexacopter_body_to_base_link" type="fixed">
-    <parent link="hexacopter_body"/>
-    <child link="base_link"/>
-    <origin xyz="0 0 0" rpy="3.14 0 0"/>
-  </joint>-->
-  <!-- Properties -->
   <xacro:property name="link_length" value="0.25"/>
   <xacro:property name="joint_radius" value="0.05"/>
@@ -16,5 +7,4 @@
   <xacro:property name="gripper_length" value="0.1"/>
   <xacro:property name="link_mass" value="1.0"/>
-<!-- World Link Definition -->
   <link name="world">
     <inertial>
@@ -24,5 +14,4 @@
     </inertial>
   </link>
-  <!-- Fixed Joint to Attach Base Link to World -->
 <joint name="base_to_world" type="fixed">
   <parent link="world"/>
@@ -30,5 +19,4 @@
   <origin xyz="0 0 0" rpy="0 0 0"/>
 </joint>
-  <!-- Base Link -->
   <link name="base_link">
     <visual>
@@ -53,5 +41,4 @@
     </inertial>
   </link>
-  <!-- Joint 1 -->
   <joint name="joint_1" type="revolute">
     <parent link="base_link"/>
@@ -62,5 +49,4 @@
     <dynamics damping="1.0" friction="1.0"/>
   </joint>
-  <!-- Link 1 -->
   <link name="link_1">
     <visual>
@@ -85,5 +71,4 @@
     </inertial>
   </link>
-  <!-- Joint 2 -->
   <joint name="joint_2" type="revolute">
     <parent link="link_1"/>
@@ -94,5 +79,4 @@
     <dynamics damping="1.0" friction="1.0"/>
   </joint>
-  <!-- Link 2 -->
   <link name="link_2">
     <visual>
@@ -117,5 +101,4 @@
     </inertial>
   </link>
-  <!-- Joint 3 -->
   <joint name="joint_3" type="revolute">
     <parent link="link_2"/>
@@ -126,5 +109,4 @@
     <dynamics damping="1.0" friction="1.0"/>
   </joint>
-  <!-- Link 3 -->
   <link name="link_3">
     <visual>
@@ -149,5 +131,4 @@
     </inertial>
   </link>
-  <!-- Gripper Joint -->
   <joint name="gripper_joint" type="revolute">
     <parent link="link_3"/>
@@ -158,5 +139,4 @@
     <dynamics damping="1.0" friction="1.0"/>
   </joint>
-  <!-- Gripper Link -->
   <link name="gripper">
     <visual>
@@ -181,5 +161,4 @@
     </inertial>
   </link>
-  <!-- Transmissions -->
   <transmission name="transmission_joint_1">
     <type>transmission_interface/SimpleTransmission</type>

File: my_hexacopter/urdf/sensors.xacro (robot description, xacro)
@@ -22,5 +22,4 @@
     </sensor>
   </gazebo>
-  <!-- Sensor Link (Depth Camera) -->
   <link name="depth_camera_link">
     <visual>
@@ -45,5 +44,4 @@
     </inertial>
   </link>
-  <!-- Fixed Joint to Attach Sensor to Robot Arm -->
   <joint name="depth_camera_joint" type="fixed">
     <parent link="hexacopter_body"/>
@@ -63,5 +61,4 @@
   </joint>
   <link name="camera_rgb_optical_frame"/>
-  <!-- Camera Sensor -->
   <gazebo reference="camera_rgb_optical_frame">
       <sensor name="camera" type="camera">
@@ -82,7 +79,4 @@
             <noise>
               <type>gaussian</type>
-              <!-- Noise is sampled independently per pixel on each frame.
-                    That pixel's noise value is added to each of its color
-                    channels, which at that point lie in the range [0,1]. -->
               <mean>0.0</mean>
               <stddev>0.007</stddev>
@@ -91,11 +85,5 @@
             <plugin name="camera_driver" filename="libgazebo_ros_camera.so">
               <ros>
-                <!-- <namespace>test_cam</namespace> -->
-                <!-- <remapping>image_raw:=image_demo</remapping> -->
-                <!-- <remapping>camera_info:=camera_info_demo</remapping> -->
               </ros>
-              <!-- camera_name>omit so it defaults to sensor name</camera_name-->
-              <!-- frame_name>omit so it defaults to link name</frameName-->
-              <!-- <hack_baseline>0.07</hack_baseline> -->
             </plugin>
         </sensor>
